File: Boards/Rev A/POV-Stick-5050 Rev A.sch (KiCad schematic (older format))
At the start: 23 parts, among them J1 ISP_Header, J2 Batt Conn, SW1 Power Switch, U1 ATTINY85-20SU, U10 APA102C, U11 APA102C, U2 APA102C, U3 APA102C, U4 APA102C, U5 APA102C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

Commit message: Created compact 5050 footprint
And I'll have to create other smaller footprints or select smaller components if I want this stick thing to look nice.
Parts:
- U10, U11, U2, U3, U4, U5, U6, U7, U8, U9: footprint LEDs:LED_RGB_5050-6 -> MyLEDs:LED_RGB_5050-6_Compact
Changed lines of the file:
@@
 F 0 "U2" H 5450 7006 60  0000 C CNN
 F 1 "APA102C" H 5600 6600 60  0000 C CNN
-F 2 "LEDs:LED_RGB_5050-6" H 5600 6600 60  0001 C CNN
+F 2 "MyLEDs:LED_RGB_5050-6_Compact" H 5600 6600 60  0001 C CNN
 F 3 "" H 5600 6600 60  0001 C CNN
 	1    5600 6650
@@
 F 0 "U3" H 6400 7006 60  0000 C CNN
 F 1 "APA102C" H 6550 6600 60  0000 C CNN
-F 2 "LEDs:LED_RGB_5050-6" H 6550 6600 60  0001 C CNN
+F 2 "MyLEDs:LED_RGB_5050-6_Compact" H 6550 6600 60  0001 C CNN
 F 3 "" H 6550 6600 60  0001 C CNN
 	1    6550 6650
@@
 F 0 "U4" H 7350 7006 60  0000 C CNN
 F 1 "APA102C" H 7500 6600 60  0000 C CNN
-F 2 "LEDs:LED_RGB_5050-6" H 7500 6600 60  0001 C CNN
+F 2 "MyLEDs:LED_RGB_5050-6_Compact" H 7500 6600 60  0001 C CNN
 F 3 "" H 7500 6600 60  0001 C CNN
 	1    7500 6650
@@
 F 0 "U5" H 8300 7006 60  0000 C CNN
 F 1 "APA102C" H 8450 6600 60  0000 C CNN
-F 2 "LEDs:LED_RGB_5050-6" H 8450 6600 60  0001 C CNN
+F 2 "MyLEDs:LED_RGB_5050-6_Compact" H 8450 6600 60  0001 C CNN
 F 3 "" H 8450 6600 60  0001 C CNN
 	1    8450 6650
@@
 F 0 "U6" H 9250 7006 60  0000 C CNN
 F 1 "APA102C" H 9400 6600 60  0000 C CNN
-F 2 "LEDs:LED_RGB_5050-6" H 9400 6600 60  0001 C CNN
+F 2 "MyLEDs:LED_RGB_5050-6_Compact" H 9400 6600 60  0001 C CNN
 F 3 "" H 9400 6600 60  0001 C CNN
 	1    9400 6650
@@
 F 0 "U7" H 10200 7006 60  0000 C CNN
 F 1 "APA102C" H 10350 6600 60  0000 C CNN
-F 2 "LEDs:LED_RGB_5050-6" H 10350 6600 60  0001 C CNN
+F 2 "MyLEDs:LED_RGB_5050-6_Compact" H 10350 6600 60  0001 C CNN
 F 3 "" H 10350 6600 60  0001 C CNN
 	1    10350 6650
@@
 F 0 "U8" H 11150 7006 60  0000 C CNN
 F 1 "APA102C" H 11300 6600 60  0000 C CNN
-F 2 "LEDs:LED_RGB_5050-6" H 11300 6600 60  0001 C CNN
+F 2 "MyLEDs:LED_RGB_5050-6_Compact" H 11300 6600 60  0001 C CNN
 F 3 "" H 11300 6600 60  0001 C CNN
 	1    11300 6650
@@
 F 0 "U9" H 12100 7006 60  0000 C CNN
 F 1 "APA102C" H 12250 6600 60  0000 C CNN
-F 2 "LEDs:LED_RGB_5050-6" H 12250 6600 60  0001 C CNN
+F 2 "MyLEDs:LED_RGB_5050-6_Compact" H 12250 6600 60  0001 C CNN
 F 3 "" H 12250 6600 60  0001 C CNN
 	1    12250 6650
@@
 F 0 "U10" H 13050 7006 60  0000 C CNN
 F 1 "APA102C" H 13200 6600 60  0000 C CNN
-F 2 "LEDs:LED_RGB_5050-6" H 13200 6600 60  0001 C CNN
+F 2 "MyLEDs:LED_RGB_5050-6_Compact" H 13200 6600 60  0001 C CNN
 F 3 "" H 13200 6600 60  0001 C CNN
 	1    13200 6650
@@
 F 0 "U11" H 14000 7006 60  0000 C CNN
 F 1 "APA102C" H 14150 6600 60  0000 C CNN
-F 2 "LEDs:LED_RGB_5050-6" H 14150 6600 60  0001 C CNN
+F 2 "MyLEDs:LED_RGB_5050-6_Compact" H 14150 6600 60  0001 C CNN
 F 3 "" H 14150 6600 60  0001 C CNN
 	1    14150 6650

Commit message: OSHPark settings, preliminary component locations
Parts:
- C2: footprint Capacitors_Tantalum_SMD:CP_Tantalum_Case-C_EIA-6032-28_Hand -> Capacitors_Tantalum_SMD:CP_Tantalum_Case-C_EIA-6032-28_Reflow
- D1: value Power LED -> Heartbeat LED
Connections:
- net +BATT: no longer D1.2 (A)
- net at U1.2 (PB3(XTAL1/CLKI/~OC1B~/ADC3/PCINT3)): now also D1.2 (A)
- no-connect marks 5 -> 4
Other:
- moved on the sheet: D1, R3
Changed lines of the file:
@@
 L GND #PWR09
 U 1 1 5A461618
-P 12900 4850
-F 0 "#PWR09" H 12900 4600 50  0001 C CNN
-F 1 "GND" H 12900 4700 50  0000 C CNN
-F 2 "" H 12900 4850 50  0001 C CNN
-F 3 "" H 12900 4850 50  0001 C CNN
-	1    12900 4850
-	1    0    0    -1
-$EndComp
-$Comp
-L +BATT #PWR010
-U 1 1 5A46164D
-P 12900 3650
-F 0 "#PWR010" H 12900 3500 50  0001 C CNN
-F 1 "+BATT" H 12900 3790 50  0000 C CNN
-F 2 "" H 12900 3650 50  0001 C CNN
-F 3 "" H 12900 3650 50  0001 C CNN
-	1    12900 3650
+P 2100 7650
+F 0 "#PWR09" H 2100 7400 50  0001 C CNN
+F 1 "GND" H 2100 7500 50  0000 C CNN
+F 2 "" H 2100 7650 50  0001 C CNN
+F 3 "" H 2100 7650 50  0001 C CNN
+	1    2100 7650
 	1    0    0    -1
 $EndComp
@@
 L R_vert R3
 U 1 1 5A49C261
-P 12900 4450
-F 0 "R3" H 13000 4550 50  0000 L CNN
-F 1 "1.5k" H 13000 4450 50  0000 L CNN
-F 2 "Resistors_SMD:R_0603_HandSoldering" V 12830 4450 50  0001 C CNN
-F 3 "" H 12900 4450 50  0001 C CNN
-F 4 "0603" H 13000 4350 50  0000 L CNN "Package Size"
-F 5 "RC0603FR-071K5L" H 13000 4250 50  0000 L CNN "MFR P/N"
-	1    12900 4450
+P 2100 7250
+F 0 "R3" H 2200 7350 50  0000 L CNN
+F 1 "1.5k" H 2200 7250 50  0000 L CNN
+F 2 "Resistors_SMD:R_0603_HandSoldering" V 2030 7250 50  0001 C CNN
+F 3 "" H 2100 7250 50  0001 C CNN
+F 4 "0603" H 2200 7150 50  0000 L CNN "Package Size"
+F 5 "RC0603FR-071K5L" H 2200 7050 50  0000 L CNN "MFR P/N"
+	1    2100 7250
 	1    0    0    -1
 $EndComp
@@
 L LED_ALT_vert D1
 U 1 1 5A4A524A
-P 12900 3950
-F 0 "D1" H 13100 4050 50  0000 C CNN
-F 1 "Power LED" H 13050 3950 50  0000 L CNN
-F 2 "LEDs:LED_0603_HandSoldering" H 13000 3950 50  0001 C CNN
-F 3 "file:///Users/durandal/Documents/Projects/KiCAD%20tutorials/ATTiny85%201%20pixel%20RGB/datasheets/Power%20LED/Osram-LS_L29K-G1J2-1-Z-datasheet.pdf" H 13100 4050 50  0001 C CNN
-F 4 "0603" H 13050 3850 50  0000 L CNN "Package Size"
-F 5 "LS L29K-G1J2-1-Z" H 13050 3750 50  0000 L CNN "MFR P/N"
-	1    12900 3950
+P 2100 6750
+F 0 "D1" H 2300 6850 50  0000 C CNN
+F 1 "Heartbeat LED" H 2250 6750 50  0000 L CNN
+F 2 "LEDs:LED_0603_HandSoldering" H 2200 6750 50  0001 C CNN
+F 3 "file:///Users/durandal/Documents/Projects/KiCAD%20tutorials/ATTiny85%201%20pixel%20RGB/datasheets/Power%20LED/Osram-LS_L29K-G1J2-1-Z-datasheet.pdf" H 2300 6850 50  0001 C CNN
+F 4 "0603" H 2250 6650 50  0000 L CNN "Package Size"
+F 5 "LS L29K-G1J2-1-Z" H 2250 6550 50  0000 L CNN "MFR P/N"
+	1    2100 6750
 	1    0    0    -1
 $EndComp
@@
 F 0 "C2" H 5750 7500 50  0000 L CNN
 F 1 "100uF" H 5750 7400 50  0000 L CNN
-F 2 "Capacitors_Tantalum_SMD:CP_Tantalum_Case-C_EIA-6032-28_Hand" H 5650 7350 50  0001 C CNN
+F 2 "Capacitors_Tantalum_SMD:CP_Tantalum_Case-C_EIA-6032-28_Reflow" H 5650 7350 50  0001 C CNN
 F 3 "" H 5660 7420 50  0001 C CNN
 F 4 "10V" H 5750 7300 50  0000 L CNN "Voltage Rating"
@@
 	1    0    0    -1
 $EndComp
-Text Notes 12450 3350 0    60   ~ 0
+Text Notes 950  6300 0    60   ~ 0
 Vf = 1.8V, 2 mA Ityp\n5V-1.8 = 3.2V\n3.2V/1.5k = 2.1 mA
 $Comp
@@
 	1    0    0    -1
 $EndComp
-NoConn ~ 3900 4400
 $Comp
 L SW_DPDT_x2_horiz SW1
@@
 	1750 2400 1750 2900
 Wire Wire Line
-	12900 4300 12900 4100
-Wire Wire Line
-	12900 3650 12900 3800
+	2100 7100 2100 6900
+Wire Wire Line
+	2100 5600 2100 6600
 Wire Wire Line
 	3800 2600 3800 6400
@@
 Connection ~ 6750 4600
 Wire Wire Line
-	12900 4650 12900 4850
+	2100 7450 2100 7650
 Wire Wire Line
 	1900 5050 1900 4950
@@
 	1    0    0    -1
 $EndComp
+Wire Wire Line
+	3900 4400 3600 4400
+Wire Wire Line
+	3600 5600 3600 4400
+Wire Wire Line
+	2100 5600 3600 5600
 $EndSCHEMATC

Commit message: Finished layout
Need to add Flamingo logo
Parts:
- J1: footprint Pin_Headers:Pin_Header_Straight_2x03_Pitch2.54mm -> MyConnectors:ISP_Header_Pogo_2x03_Pitch2.54mm
Changed lines of the file:
@@
 F 0 "J1" H 3100 2700 50  0000 C CNN
 F 1 "ISP_Header" H 3050 2600 50  0000 L CNN
-F 2 "Pin_Headers:Pin_Header_Straight_2x03_Pitch2.54mm" H 3150 2150 50  0001 C CNN
+F 2 "MyConnectors:ISP_Header_Pogo_2x03_Pitch2.54mm" H 3150 2150 50  0001 C CNN
 F 3 "" H 3150 2150 50  0001 C CNN
 F 4 "N/S, pogo pin" H 3050 2200 50  0000 L CNN "PN"

Commit message: Added text "wrong footprint" for aTtINY85
Other:
- note added: "WRONG FOOTPRINT\n"
Changed lines of the file:
@@
 Wire Wire Line
 	2100 5600 3600 5600
+Text Notes 4650 3850 0    60   ~ 0
+WRONG FOOTPRINT\n
 $EndSCHEMATC
